Commit message: 1. Moved k_eff from params to reference 2. Increased friction params (not sure if needed, we can reduce them later) 3. Removed limits on effort (once again, we can restore them later) 4. Removed pause flag (still need to fix the startup pose bug) Signed-off-by: Darpa Tech 3 <darpa3@SMILe03.(none)>

File: gcb_description/urdf/gcb.xacro (robot description, xacro)
@@ -200,5 +200,5 @@
     <child link="right_leg"/>
     <dynamics damping="0.1" friction="0.0"/>
-    <limit effort="220" lower="-1.57" upper="1.57" velocity="12"/>
+    <limit effort="2000" lower="-1.57" upper="1.57" velocity="12"/>
     <safety_controller k_position="100" k_velocity="10" soft_lower_limit="-1.47" soft_upper_limit="1.47"/>
   </joint>
@@ -209,5 +209,5 @@
     <child link="left_talus"/>
     <dynamics damping="0.1" friction="0.0"/>
-    <limit effort="220" lower="-1.65" upper="1.3" velocity="12"/>
+    <limit effort="2000" lower="-1.65" upper="1.3" velocity="12"/>
     <safety_controller k_position="100" k_velocity="10" soft_lower_limit="-1.55" soft_upper_limit="1.2"/>
   </joint>
@@ -223,5 +223,5 @@
     <child link="right_talus"/>
     <dynamics damping="0.1" friction="0.0"/>
-    <limit effort="220" lower="-1.65" upper="1.3" velocity="12"/>
+    <limit effort="2000" lower="-1.65" upper="1.3" velocity="12"/>
     <safety_controller k_position="100" k_velocity="10" soft_lower_limit="-1.55" soft_upper_limit="1.2"/>
   </joint>
